File: PCB/Drivers_PCB.kicad_sch (KiCad schematic)
At the start: 30 parts, among them J1 Power_Connector, J10 Conn_01x08, J2 Fan_Connector, J3 Motor_1_connector, J4 EOC_Switch_Connector, J5 Motor_2_connector, J6 IR_LED_Connector, J7 Conn_01x08, J8 Conn_01x06, J9 Conn_01x10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

Commit message: Fixing the shield pins matching
Connections:
- net DIR1: now also J10.7 (Pin_7); no longer J10.2 (Pin_2)
- net DIR2: now also J10.8 (Pin_8); no longer J10.1 (Pin_1)
- net GND: now also J9.7 (Pin_7); no longer J9.4 (Pin_4)
- net IR_LED: now also J9.5 (Pin_5); no longer J9.6 (Pin_6)
- net MS1: now also J9.1 (Pin_1); no longer J9.10 (Pin_10)
- net MS2: now also J9.2 (Pin_2); no longer J9.9 (Pin_9)
- net MS3: now also J9.3 (Pin_3); no longer J9.8 (Pin_8)
- net RESET1: now also J10.5 (Pin_5); no longer J10.4 (Pin_4)
- net RESET2: now also J10.6 (Pin_6); no longer J10.3 (Pin_3)
- net SLEEP1: now also J10.3 (Pin_3); no longer J10.6 (Pin_6)
- net SLEEP2: now also J10.4 (Pin_4); no longer J10.5 (Pin_5)
- net STEP1: now also J9.4 (Pin_4); no longer J9.7 (Pin_7)
- net STEP2: now also J9.6 (Pin_6); no longer J9.5 (Pin_5)
Changed lines of the file:
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@@
+	)
+	(symbol
+		(lib_id "Connector_Generic:Conn_01x08")
+		(at 207.01 68.58 0)
+		(mirror x)
+		(unit 1)
+		(exclude_from_sim no)
+		(in_bom yes)
+		(on_board yes)
+		(dnp no)
+		(property "Reference" "J10"
+			(at 209.55 68.5801 0)
+			(effects
+				(font
+					(size 1.27 1.27)
+				)
+				(justify left)
+			)
+		)
+		(property "Value" "Conn_01x08"
+			(at 209.55 66.0401 0)
+			(effects
+				(font
+					(size 1.27 1.27)
+				)
+				(justify left)
+			)
+		)
+		(property "Footprint" "Connector_PinHeader_2.54mm:PinHeader_1x08_P2.54mm_Vertical"
+			(at 207.01 68.58 0)
+			(effects
+				(font
+					(size 1.27 1.27)
+				)
+				(hide yes)
+			)
+		)
+		(property "Datasheet" "~"
+			(at 207.01 68.58 0)
+			(effects
+				(font
+					(size 1.27 1.27)
+				)
+				(hide yes)
+			)
+		)
+		(property "Description" "Generic connector, single row, 01x08, script generated (kicad-library-utils/schlib/autogen/connector/)"
+			(at 207.01 68.58 0)
+			(effects
+				(font
+					(size 1.27 1.27)
+				)
+				(hide yes)
+			)
+		)
+		(pin "4"
+		)
+		(pin "3"
+		)
+		(pin "2"
+		)
+		(pin "6"
+		)
+		(pin "1"
+		)
+		(pin "8"
+		)
+		(pin "5"
+		)
+		(pin "7"
+		)
+		(instances
+			(project "Drivers_PCB"
+				(path "/965d1d26-667e-4a58-b302-d26df24cf4f3"
+					(reference "J10")
+					(unit 1)
+				)
+			)
+		)
 	)
 	(symbol
@@
 	)
 	(symbol
-		(lib_id "Connector_Generic:Conn_01x10")
-		(at 207.01 40.64 0)
-		(unit 1)
-		(exclude_from_sim no)
-		(in_bom yes)
-		(on_board yes)
-		(dnp no)
-		(fields_autoplaced yes)
-		(property "Reference" "J9"
-			(at 209.55 40.6399 0)
-			(effects
-				(font
-					(size 1.27 1.27)
-				)
-				(justify left)
-			)
-		)
-		(property "Value" "Conn_01x10"
-			(at 209.55 43.1799 0)
-			(effects
-				(font
-					(size 1.27 1.27)
-				)
-				(justify left)
-			)
-		)
-		(property "Footprint" "Connector_PinHeader_2.54mm:PinHeader_1x10_P2.54mm_Vertical"
-			(at 207.01 40.64 0)
-			(effects
-				(font
-					(size 1.27 1.27)
-				)
-				(hide yes)
-			)
-		)
-		(property "Datasheet" "~"
-			(at 207.01 40.64 0)
-			(effects
-				(font
-					(size 1.27 1.27)
-				)
-				(hide yes)
-			)
-		)
-		(property "Description" "Generic connector, single row, 01x10, script generated (kicad-library-utils/schlib/autogen/connector/)"
-			(at 207.01 40.64 0)
-			(effects
-				(font
-					(size 1.27 1.27)
-				)
-				(hide yes)
-			)
-		)
-		(pin "6"
-		)
-		(pin "5"
-		)
-		(pin "8"
-		)
-		(pin "1"
-		)
-		(pin "10"
-		)
-		(pin "2"
-		)
-		(pin "3"
-		)
-		(pin "4"
-		)
-		(pin "7"
-		)
-		(pin "9"
-		)
-		(instances
-			(project ""
-				(path "/965d1d26-667e-4a58-b302-d26df24cf4f3"
-					(reference "J9")
-					(unit 1)
-				)
-			)
-		)
-	)
-	(symbol
 		(lib_id "Device:C_Small")
 		(at 236.22 104.14 270)
@@
 	)
 	(symbol
-		(lib_id "Connector_Generic:Conn_01x08")
-		(at 207.01 66.04 0)
-		(unit 1)
-		(exclude_from_sim no)
-		(in_bom yes)
-		(on_board yes)
-		(dnp no)
-		(fields_autoplaced yes)
-		(property "Reference" "J10"
-			(at 209.55 66.0399 0)
-			(effects
-				(font
-					(size 1.27 1.27)
-				)
-				(justify left)
-			)
-		)
-		(property "Value" "Conn_01x08"
-			(at 209.55 68.5799 0)
-			(effects
-				(font
-					(size 1.27 1.27)
-				)
-				(justify left)
-			)
-		)
-		(property "Footprint" "Connector_PinHeader_2.54mm:PinHeader_1x08_P2.54mm_Vertical"
-			(at 207.01 66.04 0)
-			(effects
-				(font
-					(size 1.27 1.27)
-				)
-				(hide yes)
-			)
-		)
-		(property "Datasheet" "~"
-			(at 207.01 66.04 0)
-			(effects
-				(font
-					(size 1.27 1.27)
-				)
-				(hide yes)
-			)
-		)
-		(property "Description" "Generic connector, single row, 01x08, script generated (kicad-library-utils/schlib/autogen/connector/)"
-			(at 207.01 66.04 0)
-			(effects
-				(font
-					(size 1.27 1.27)
-				)
-				(hide yes)
-			)
-		)
-		(pin "4"
-		)
-		(pin "3"
-		)
-		(pin "2"
-		)
-		(pin "6"
-		)
-		(pin "1"
-		)
-		(pin "8"
-		)
-		(pin "5"
-		)
-		(pin "7"
-		)
-		(instances
-			(project "Drivers_PCB"
-				(path "/965d1d26-667e-4a58-b302-d26df24cf4f3"
-					(reference "J10")
-					(unit 1)
-				)
-			)
-		)
-	)
-	(symbol
 		(lib_id "Connector_Generic:Conn_01x03")
 		(at 116.84 40.64 0)
@@
 					(unit 1)
 				)
+			)
+		)
+	)
+	(symbol
+		(lib_id "Connector_Generic:Conn_01x10")
+		(at 207.01 43.18 0)
+		(mirror x)
+		(unit 1)
+		(exclude_from_sim no)
+		(in_bom yes)
+		(on_board yes)
+		(dnp no)
+		(property "Reference" "J9"
+			(at 209.55 43.1801 0)
+			(effects
+				(font
+					(size 1.27 1.27)
+				)
+				(justify left)
+			)
+		)
+		(property "Value" "Conn_01x10"
+			(at 209.55 40.6401 0)
+			(effects
+				(font
+					(size 1.27 1.27)
+				)
+				(justify left)
+			)
+		)
+		(property "Footprint" "Connector_PinHeader_2.54mm:PinHeader_1x10_P2.54mm_Vertical"
+			(at 207.01 43.18 0)
+			(effects
+				(font
+					(size 1.27 1.27)
+				)
+				(hide yes)
+			)
+		)
+		(property "Datasheet" "~"
+			(at 207.01 43.18 0)
+			(effects
+				(font
+					(size 1.27 1.27)
+				)
+				(hide yes)
+			)
+		)
+		(property "Description" "Generic connector, single row, 01x10, script generated (kicad-library-utils/schlib/autogen/connector/)"
+			(at 207.01 43.18 0)
+			(effects
+				(font
+					(size 1.27 1.27)
+				)
+				(hide yes)
+			)
+		)
+		(pin "6"
+		)
+		(pin "5"
+		)
+		(pin "8"
+		)
+		(pin "1"
+		)
+		(pin "10"
+		)
+		(pin "2"
+		)
+		(pin "3"
+		)
+		(pin "4"
+		)
+		(pin "7"
+		)
+		(pin "9"
+		)
+		(instances
+			(project "Drivers_PCB"
+				(path "/965d1d26-667e-4a58-b302-d26df24cf4f3"
+					(reference "J9")
+					(unit 1)
+				)

Commit message: Cleaning the git
Parts:
- added J11: SWITCH_Connector, Connector_JST:JST_XH_B2B-XH-A_1x02_P2.50mm_Vertical, symbol Connector_Generic:Conn_01x02
Connections:
- net VBB: now also J11.1 (Pin_1); no longer J1.1 (Pin_1)
- new net: J1.1 (Pin_1), J11.2 (Pin_2)
Other:
- moved on the sheet: J1
Changed lines of the file:
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@@
 	)
 	(junction
-		(at 46.99 49.53)
-		(diameter 0)
-		(color 0 0 0 0)
-	)
-	(junction
 		(at 128.27 160.02)
 		(diameter 0)
@@
 	)
 	(junction
+		(at 62.23 49.53)
+		(diameter 0)
+		(color 0 0 0 0)
+	)
+	(junction
 		(at 265.43 114.3)
 		(diameter 0)
@@
 	(wire
 		(pts
-			(xy 168.91 114.3) (xy 168.91 116.84)
+			(xy 62.23 49.53) (xy 63.5 49.53)
 		)
 		(stroke
@@
 	(wire
 		(pts
-			(xy 273.05 142.24) (xy 273.05 127)
+			(xy 168.91 114.3) (xy 168.91 116.84)
 		)
 		(stroke
@@
 	(wire
 		(pts
-			(xy 121.92 160.02) (xy 128.27 160.02)
+			(xy 273.05 142.24) (xy 273.05 127)
 		)
 		(stroke
@@
 	(wire
 		(pts
-			(xy 265.43 118.11) (xy 259.08 118.11)
+			(xy 121.92 160.02) (xy 128.27 160.02)
 		)
 		(stroke
@@
 	(wire
 		(pts
-			(xy 168.91 142.24) (xy 173.99 142.24)
+			(xy 265.43 118.11) (xy 259.08 118.11)
 		)
 		(stroke
@@
 	(wire
 		(pts
-			(xy 154.94 127) (xy 158.75 127)
+			(xy 168.91 142.24) (xy 173.99 142.24)
 		)
 		(stroke
@@
 	(wire
 		(pts
-			(xy 116.84 99.06) (xy 121.92 99.06)
+			(xy 154.94 127) (xy 158.75 127)
 		)
 		(stroke
@@
 	(wire
 		(pts
-			(xy 45.72 49.53) (xy 46.99 49.53)
+			(xy 116.84 99.06) (xy 121.92 99.06)
 		)
 		(stroke
@@
 	(wire
 		(pts
+			(xy 53.34 49.53) (xy 53.34 45.72)
+		)
+		(stroke
+			(width 0)
+			(type default)
+		)
+	)
+	(wire
+		(pts
 			(xy 121.92 99.06) (xy 121.92 101.6)
 		)
@@
 	(wire
 		(pts
+			(xy 55.88 49.53) (xy 62.23 49.53)
+		)
+		(stroke
+			(width 0)
+			(type default)
+		)
+	)
+	(wire
+		(pts
 			(xy 220.98 99.06) (xy 226.06 99.06)
 		)
@@
 	(wire
 		(pts
-			(xy 46.99 49.53) (xy 48.26 49.53)
+			(xy 97.79 114.3) (xy 104.14 114.3)
 		)
 		(stroke
@@
 	(wire
 		(pts
-			(xy 97.79 114.3) (xy 104.14 114.3)
+			(xy 265.43 114.3) (xy 273.05 114.3)
 		)
 		(stroke
@@
 	(wire
 		(pts
-			(xy 265.43 114.3) (xy 273.05 114.3)
+			(xy 128.27 157.48) (xy 128.27 160.02)
 		)
 		(stroke
@@
 	(wire
 		(pts
-			(xy 128.27 157.48) (xy 128.27 160.02)
+			(xy 55.88 45.72) (xy 55.88 49.53)
 		)
 		(stroke
@@
 	(wire
 		(pts
-			(xy 45.72 52.07) (xy 48.26 52.07)
+			(xy 45.72 52.07) (xy 63.5 52.07)
 		)
 		(stroke
@@
 	(wire
 		(pts
+			(xy 45.72 49.53) (xy 53.34 49.53)
+		)
+		(stroke
+			(width 0)
+			(type default)
+		)
+	)
+	(wire
+		(pts
 			(xy 259.08 127) (xy 262.89 127)
 		)
@@
 	(symbol
 		(lib_id "Connector_Generic:Conn_01x02")
-		(at 53.34 49.53 0)
+		(at 68.58 49.53 0)
 		(unit 1)
 		(exclude_from_sim no)
@@
 		(fields_autoplaced yes)
 		(property "Reference" "J1"
-			(at 55.88 49.5299 0)
+			(at 71.12 49.5299 0)
 			(effects
 				(font
@@
 		)
 		(property "Value" "Power_Connector"
-			(at 55.88 52.0699 0)
+			(at 71.12 52.0699 0)
 			(effects
 				(font
@@
 		)
 		(property "Footprint" "TerminalBlock:TerminalBlock_bornier-2_P5.08mm"
-			(at 53.34 49.53 0)
+			(at 68.58 49.53 0)
 			(effects
 				(font
@@
 		)
 		(property "Datasheet" "~"
-			(at 53.34 49.53 0)
+			(at 68.58 49.53 0)
 			(effects
 				(font
@@
 		)
 		(property "Description" "Generic connector, single row, 01x02, script generated (kicad-library-utils/schlib/autogen/connector/)"
-			(at 53.34 49.53 0)
+			(at 68.58 49.53 0)
 			(effects
 				(font
@@
 	(symbol
 		(lib_id "power:PWR_FLAG")
-		(at 46.99 49.53 0)
+		(at 62.23 49.53 0)
 		(unit 1)
 		(exclude_from_sim no)
@@
 		(fields_autoplaced yes)
 		(property "Reference" "#FLG01"
-			(at 46.99 47.625 0)
+			(at 62.23 47.625 0)
 			(effects
 				(font
@@
 		)
 		(property "Value" "PWR_FLAG"
-			(at 46.99 44.45 0)
+			(at 62.23 44.45 0)
 			(effects
 				(font
@@
 		)
 		(property "Footprint" ""
-			(at 46.99 49.53 0)
+			(at 62.23 49.53 0)
 			(effects
 				(font
@@
 		)
 		(property "Datasheet" "~"
-			(at 46.99 49.53 0)
+			(at 62.23 49.53 0)
 			(effects
 				(font
@@
 		)
 		(property "Description" "Special symbol for telling ERC where power comes from"
-			(at 46.99 49.53 0)
+			(at 62.23 49.53 0)
 			(effects
 				(font
@@
 					(unit 1)
 				)
+			)
+		)
+	)
+	(symbol
+		(lib_id "Connector_Generic:Conn_01x02")
+		(at 53.34 40.64 90)
+		(unit 1)
+		(exclude_from_sim no)
+		(in_bom yes)
+		(on_board yes)
+		(dnp no)
+		(fields_autoplaced yes)
+		(property "Reference" "J11"
+			(at 58.42 39.3699 90)
+			(effects
+				(font
+					(size 1.27 1.27)
+				)
+				(justify right)
+			)
+		)
+		(property "Value" "SWITCH_Connector"
+			(at 58.42 41.9099 90)
+			(effects
+				(font
+					(size 1.27 1.27)
+				)
+				(justify right)
+			)
+		)
+		(property "Footprint" "Connector_JST:JST_XH_B2B-XH-A_1x02_P2.50mm_Vertical"
+			(at 53.34 40.64 0)
+			(effects
+				(font
+					(size 1.27 1.27)
+				)
+				(hide yes)
+			)
+		)
+		(property "Datasheet" "~"
+			(at 53.34 40.64 0)
+			(effects
+				(font
+					(size 1.27 1.27)
+				)
+				(hide yes)
+			)
+		)
+		(property "Description" "Generic connector, single row, 01x02, script generated (kicad-library-utils/schlib/autogen/connector/)"
+			(at 53.34 40.64 0)
+			(effects
+				(font
+					(size 1.27 1.27)
+				)
+				(hide yes)
+			)
+		)
+		(pin "1"
+		)
+		(pin "2"
+		)
+		(instances
+			(project "Drivers_PCB"
+				(path "/965d1d26-667e-4a58-b302-d26df24cf4f3"
+					(reference "J11")
+					(unit 1)
+				)
