File: PCB/Drivers_PCB.kicad_sch (KiCad schematic)
At the start: 31 parts, among them J1 Power_Connector, J10 Conn_01x08, J11 SWITCH_Connector, J2 Fan_Connector, J3 Motor_1_connector, J4 EOC_Switch_Connector, J5 Motor_2_connector, J6 IR_LED_Connector, J7 Conn_01x08, J8 Conn_01x06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

Commit message: filling in all components values
Parts:
- R1, R5: value R_Small -> 5k
- R2: value R_Small -> 20k
- R3, R4, R7, R8: value R_Small -> 0.5
- R6: value ~ -> 20k
Changed lines of the file:
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@@
 			)
 		)
-		(property "Value" "R_Small"
+		(property "Value" "0.5"
 			(at 161.544 132.588 90)
 			(effects
@@
 					(size 1.27 1.27)
 				)
-				(hide yes)
 			)
 		)
@@
 			)
 		)
-		(property "Value" "R_Small"
+		(property "Value" "0.5"
 			(at 265.684 132.588 90)
 			(effects
@@
 					(size 1.27 1.27)
 				)
-				(hide yes)
 			)
 		)
@@
 		(fields_autoplaced yes)
 		(property "Reference" "R1"
-			(at 100.33 115.5699 0)
-			(effects
-				(font
-					(size 1.27 1.27)
-				)
-				(justify left)
-			)
-		)
-		(property "Value" "R_Small"
+			(at 100.33 116.8399 0)
+			(effects
+				(font
+					(size 1.27 1.27)
+				)
+				(justify left)
+			)
+		)
+		(property "Value" "5k"
 			(at 100.33 118.1099 0)
 			(effects
@@
 				)
 				(justify left)
-				(hide yes)
 			)
 		)
@@
 			)
 		)
-		(property "Value" "~"
-			(at 222.758 97.282 0)
-			(effects
-				(font
-					(size 1.27 1.27)
-				)
-				(justify left)
-				(hide yes)
+		(property "Value" "20k"
+			(at 227.076 106.426 0)
+			(effects
+				(font
+					(size 1.27 1.27)
+				)
+				(justify left)
 			)
 		)
@@
 			)
 		)
-		(property "Value" "R_Small"
+		(property "Value" "0.5"
 			(at 161.29 147.574 90)
 			(effects
@@
 					(size 1.27 1.27)
 				)
-				(hide yes)
 			)
 		)
@@
 			)
 		)
-		(property "Value" "R_Small"
+		(property "Value" "5k"
 			(at 204.47 118.1099 0)
 			(effects
@@
 				)
 				(justify left)
-				(hide yes)
 			)
 		)
@@
 			)
 		)
-		(property "Value" "R_Small"
-			(at 118.618 97.282 0)
-			(effects
-				(font
-					(size 1.27 1.27)
-				)
-				(justify left)
-				(hide yes)
+		(property "Value" "20k"
+			(at 123.19 106.172 0)
+			(effects
+				(font
+					(size 1.27 1.27)
+				)
+				(justify left)
 			)
 		)
@@
 			)
 		)
-		(property "Value" "R_Small"
+		(property "Value" "0.5"
 			(at 265.43 147.574 90)
 			(effects
@@
 					(size 1.27 1.27)
 				)
-				(hide yes)
-			)
-		)
+			)
+		)
