File: PCB/Drivers_PCB.kicad_pcb (KiCad board)
At the start: 4 copper layers, 54 x 51 mm, 33 parts, among them J1 Power_Connector, J10 Conn_01x08, J11 SWITCH_Connector, J2 Fan_Connector, J3 Motor_1_connector, J4 EOC_Switch_Connector, J5 Motor_2_connector, J6 IR_LED_Connector, J7 Conn_01x08, J8 Conn_01x06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

Commit message: updating useless files
Parts:
- R1, R5: value R_Small -> 5k
- R2: value R_Small -> 20k
- R3, R4, R7, R8: value R_Small -> 0.5
- R6: value ~ -> 20k
Changed lines of the file:
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@@
 			)
 		)
-		(property "Value" "R_Small"
+		(property "Value" "0.5"
 			(at 0 1.65 0)
 			(layer "F.Fab")
@@
 			)
 		)
-		(property "Value" "~"
+		(property "Value" "20k"
 			(at 0 1.65 0)
 			(layer "F.Fab")
@@
 			)
 		)
-		(property "Value" "R_Small"
+		(property "Value" "5k"
 			(at 0 1.65 0)
 			(layer "F.Fab")
@@
 			)
 		)
-		(property "Value" "R_Small"
+		(property "Value" "0.5"
 			(at 0 1.65 0)
 			(layer "F.Fab")
@@
 			)
 		)
-		(property "Value" "R_Small"
+		(property "Value" "20k"
 			(at 0 1.65 0)
 			(layer "F.Fab")
@@
 			)
 		)
-		(property "Value" "R_Small"
+		(property "Value" "0.5"
 			(at 0 1.65 0)
 			(layer "F.Fab")
@@
 			)
 		)
-		(property "Value" "R_Small"
+		(property "Value" "5k"
 			(at 0 1.65 0)
 			(layer "F.Fab")
@@
 			)
 		)
-		(property "Value" "R_Small"
+		(property "Value" "0.5"
 			(at 0 1.65 0)
 			(layer "F.Fab")
